Commit message: Fix naming

File: robot_project/urdf/robot.urdf (robot description, URDF)
Before this commit: robot robot, 5 links, 4 joints
Links:
- link link_chassis: geometry collision mesh filename=package://robot_project/meshes/chassis.stl; visual mesh filename=package://robot_project/meshes/chassis.stl
- link link_left_wheel: geometry collision cylinder length=0.12 radius=0.08; collision cylinder length=0.12 radius=0.4
- link link_right_wheel: geometry collision cylinder length=0.12 radius=0.08; collision cylinder length=0.12 radius=0.4
