Commit message: Removed extra code

File: robot_project/urdf/robot.xacro (robot description, xacro)
@@ -10,7 +10,4 @@
         </inertial>
         <collision>
-            <!-- <geometry>
-                <box size="2 1.3 0.4" />
-            </geometry> -->
             <geometry>
                 <mesh filename="package://robot_project/meshes/chassis.stl" />
@@ -21,7 +18,4 @@
                 <mesh filename="package://robot_project/meshes/chassis.stl" />
             </geometry>
-            <!-- <geometry>
-                <box size="2 1.3 0.4" />
-            </geometry> -->
             <material name="DarkBlue">
                 <color rgba="0.2 0.2 0.4 1" />
