Commit message: Updated robot

File: robot_project/urdf/gazebo.xacro (robot description, xacro)
@@ -5,18 +5,23 @@
         <material>Gazebo/Blue</material>
     </gazebo>
-    <gazebo reference="link_caster_wheel">
-        <material>Gazebo/Grey</material>
-        <mu1>0</mu1>
-        <mu2>0</mu2>
-    </gazebo>
-    <gazebo reference="link_left_wheel">
+    <gazebo reference="link_left_back_wheel">
         <material>Gazebo/Black</material>
         <mu1>1</mu1>
         <mu2>1</mu2>
     </gazebo>
-    <gazebo reference="link_right_wheel">
+    <gazebo reference="link_right_back_wheel">
         <material>Gazebo/Black</material>
         <mu1>1</mu1>
         <mu2>1</mu2>
+    </gazebo>
+    <gazebo reference="link_left_front_wheel">
+        <material>Gazebo/Black</material>
+        <mu1>0</mu1>
+        <mu2>0</mu2>
+    </gazebo>
+    <gazebo reference="link_right_front_wheel">
+        <material>Gazebo/Black</material>
+        <mu1>0</mu1>
+        <mu2>0</mu2>
     </gazebo>
     <gazebo reference="joint_chassis_caster_wheel">
@@ -27,6 +32,6 @@
             <alwaysOn>true</alwaysOn>
             <updateRate>20</updateRate>
-            <leftJoint>joint_chassis_left_wheel</leftJoint>
-            <rightJoint>joint_chassis_right_wheel</rightJoint>
+            <leftJoint>joint_chassis_left_back_wheel</leftJoint>
+            <rightJoint>joint_chassis_right_back_wheel</rightJoint>
             <wheelSeparation>1.66</wheelSeparation>
             <wheelDiameter>0.8</wheelDiameter>

File: robot_project/urdf/robot.xacro (robot description, xacro)
@@ -2,4 +2,17 @@
 <robot name="robot" xmlns:xacro="http://www.ros.org/wiki/xacro">
     <xacro:include filename="$(find robot_project)/urdf/gazebo.xacro" />
+ <!-- Parameters -->
+    <xacro:property name="chassis_mass" value="10" />
+    <xacro:property name="radius_wheel" value="0.15" />
+    <xacro:property name="length_wheel" value="0.12" />
+    <xacro:property name="radius_cylinder_wheel" value="0.04" />
+    <xacro:property name="length_cylinder_wheel" value="0.12" />
+    <!-- Gazebo tags - Laser scan -->
+    <gazebo reference="joint_laser_scan_chassis">
+        <preserveFixedJoint>true</preserveFixedJoint>
+    </gazebo>
+    <gazebo reference="link_laser_scan">
+        <material>Gazebo/DarkGrey</material>
+    </gazebo>
     <!-- Link - chassis -->
     <link name="link_chassis">
@@ -11,10 +24,10 @@
         <collision>
             <geometry>
-                <mesh filename="package://robot_project/meshes/chassis.stl" />
-            </geometry>
-        </collision>
-        <visual>
-            <geometry>
-                <mesh filename="package://robot_project/meshes/chassis.stl" />
+                <box size="1 0.6 0.2" />
+            </geometry>
+        </collision>
+        <visual>
+            <geometry>
+                <box size="1 0.6 0.2" />
             </geometry>
             <material name="DarkBlue">
@@ -23,166 +36,181 @@
         </visual>
     </link>
-    <!-- Joint - caster wheel -->
-    <joint name="joint_chassis_caster_wheel" type="fixed">
-        <origin rpy="0 0 0" xyz="0.8 0 -0.15" />
-        <child link="link_caster_wheel" />
-        <parent link="link_chassis" />
-        <joint_properties damping="1.0" friction="1.0" />
-    </joint>
-    <!-- Link - caster wheel -->
-    <link name="link_caster_wheel">
-        <inertial>
-            <mass value="1" />
-            <origin xyz="0 0 0" rpy="0 0 0" />
-            <inertia ixx="0.002526666666667" ixy="0" ixz="0" iyy="0.002526666666667" iyz="0" izz="0.005"/>
-        </inertial>
-        <!-- Caster wheel support -->
-        <collision>
-            <origin rpy="0 0 0" xyz="0 0 -0.03" />
-            <geometry>
-                <sphere radius="0.2" />
-            </geometry>
-        </collision>
-        <visual>
-            <origin rpy="0 0 0" xyz="0 0 -0.03" />
-            <geometry>
-                <sphere radius="0.2" />
-            </geometry>
-            <material name="DarkBlue">
-                <color rgba="0.2 0.2 0.4 1" />
-            </material>
-        </visual>
-        <!-- Caster wheel -->
-        <collision>
-            <origin rpy="0 0 0" xyz="0 0 -0.15" />
-            <geometry>
-                <sphere radius="0.10" />
-            </geometry>
-        </collision>
-        <visual>
-            <origin rpy="0 0 0" xyz="0 0 -0.15" />
-            <geometry>
-                <sphere radius="0.10" />
-            </geometry>
-            <material name="Grey">
-                <color rgba="0.6 0.6 0.6 1" />
-            </material>
-        </visual>
-    </link>
-    <!-- Joint - chassis / left wheel -->
-    <joint name="joint_chassis_left_wheel" type="continuous">
-        <origin rpy="0 0 0" xyz="-0.5 0.65 0" />
-        <child link="link_left_wheel" />
-        <parent link="link_chassis" />
-        <axis rpy="0 0 0" xyz="0 1 0" />
-        <limit effort="10000" velocity="1000" />
-        <joint_properties damping="1.0" friction="1.0" />
-    </joint>
-    <!-- Link - left wheel -->
-    <link name="link_left_wheel">
-        <inertial>
-            <mass value="1" />
-            <origin xyz="0 0 0" rpy="0 0 0" />
-            <inertia ixx="0.002526666666667" ixy="0" ixz="0" iyy="0.002526666666667" iyz="0" izz="0.005"/>
-        </inertial>
-        <!-- Tires -->
-        <collision>
-            <origin rpy="1.5707 0 0" xyz="0 0.18 0" />
-            <geometry>
-                <cylinder length="0.12" radius="0.4"/>
-            </geometry>
-        </collision>
-        <visual>
-            <origin rpy="1.5707 0 0" xyz="0 0.18 0" />
-            <geometry>
-                <mesh filename="package://robot_project/meshes/wheel.stl" />
-            </geometry>
-            <material name="Black">
-                <color rgba="0.1 0.1 0.1 1" />
-            </material>
-        </visual>
-        <!-- Axle -->
-        <collision>
-            <origin rpy="1.5707 0 0" xyz="0 0.06 0" />
-            <geometry>
-                <cylinder length="0.12" radius="0.08"/>
-            </geometry>
-        </collision>
-        <visual>
-            <origin rpy="1.5707 0 0" xyz="0 0.06 0" />
-            <geometry>
-                <cylinder length="0.12" radius="0.08"/>
-            </geometry>
-            <material name="Grey">
-                <color rgba="0.6 0.6 0.6 1" />
-            </material>
-        </visual>
-        <!-- Hubcap -->
-        <visual>
-            <origin rpy="1.5707 0 0" xyz="0 0.18 0" />
-            <geometry>
-                <box size="0.02 0.5 0.02" />
-            </geometry>
-            <material name="Grey">
-                <color rgba="0.6 0.6 0.6 1" />
-            </material>
-        </visual>
-    </link>
-    <!-- Joint - chassis / right wheel -->
-    <joint name="joint_chassis_right_wheel" type="continuous">
-        <origin rpy="0 0 0" xyz="-0.5 -0.65 0" />
-        <child link="link_right_wheel" />
-        <parent link="link_chassis" />
-        <axis rpy="0 0 0" xyz="0 1 0" />
-        <limit effort="10000" velocity="1000" />
-        <joint_properties damping="1.0" friction="1.0" />
-    </joint>
-    <!-- Link - right wheel -->
-    <link name="link_right_wheel">
-        <inertial>
-            <mass value="1" />
-            <origin xyz="0 0 0" rpy="0 0 0" />
-            <inertia ixx="0.002526666666667" ixy="0" ixz="0" iyy="0.002526666666667" iyz="0" izz="0.005"/>
-        </inertial>
-        <!-- Tires -->
-        <collision>
-            <origin rpy="1.5707 0 0" xyz="0 -0.18 0" />
-            <geometry>
-                <cylinder length="0.12" radius="0.4"/>
-            </geometry>
-        </collision>
-        <visual>
-            <origin rpy="1.5707 0 0" xyz="0 -0.18 0" />
-            <geometry>
-                <mesh filename="package://robot_project/meshes/wheel.stl" />
-            </geometry>
-            <material name="Black">
-                <color rgba="0.1 0.1 0.1 1" />
-            </material>
-        </visual>
-        <!-- Axle -->
-        <collision>
-            <origin rpy="1.5707 0 0" xyz="0 -0.06 0" />
-            <geometry>
-                <cylinder length="0.12" radius="0.08"/>
-            </geometry>
-        </collision>
-        <visual>
-            <origin rpy="1.5707 0 0" xyz="0 -0.06 0" />
-            <geometry>
-                <cylinder length="0.12" radius="0.08"/>
-            </geometry>
-            <material name="Grey">
-                <color rgba="0.6 0.6 0.6 1" />
-            </material>
-        </visual>
-        <!-- Hubcap -->
-        <visual>
-            <origin rpy="1.5707 0 0" xyz="0 -0.18 0" />
-            <geometry>
-                <box size="0.02 0.5 0.02" />
-            </geometry>
-            <material name="Grey">
-                <color rgba="0.6 0.6 0.6 1" />
+    <joint name="joint_chassis_left_back_wheel" type="continuous">
+        <origin rpy="0 0 0" xyz="-0.45 0.28 0" />
+        <child link="link_left_back_wheel" />
+        <parent link="link_chassis" />
+        <axis rpy="0 0 0" xyz="0 1 0" />
+        <limit effort="10000" velocity="1000" />
+        <joint_properties damping="1.0" friction="1.0" />
+    </joint>
+    <link name="link_left_back_wheel">
+        <inertial>
+            <mass value="1" />
+            <origin xyz="0 0 0" rpy="0 0 0" />
+            <inertia ixx="0.002526666666667" ixy="0" ixz="0" iyy="0.002526666666667" iyz="0" izz="0.005"/>
+        </inertial>
+        <collision>
+            <origin rpy="1.5707 0 0" xyz="0 0.18 0" />
+            <geometry>
+                <cylinder length="${length_wheel}" radius="${radius_wheel}"/>
+            </geometry>
+        </collision>
+        <visual>
+            <origin rpy="1.5707 0 0" xyz="0 0.18 0" />
+            <geometry>
+                <cylinder length="${length_wheel}" radius="${radius_wheel}"/>
+            </geometry>
+            <material name="Black">
+                <color rgba="0.1 0.1 0.1 1" />
+            </material>
+        </visual>
+        <collision>
+            <origin rpy="1.5707 0 0" xyz="0 0.06 0" />
+            <geometry>
+                <cylinder length="${length_cylinder_wheel}" radius="${radius_cylinder_wheel}"/>
+            </geometry>
+        </collision>
+        <visual>
+            <origin rpy="1.5707 0 0" xyz="0 0.06 0" />
+            <geometry>
+                <cylinder length="${length_cylinder_wheel}" radius="${radius_cylinder_wheel}"/>
+            </geometry>
+            <material name="Black">
+                <color rgba="0.1 0.1 0.1 1" />
+            </material>
+        </visual>
+    </link>
+    <joint name="joint_chassis_right_back_wheel" type="continuous">
+        <origin rpy="0 0 0" xyz="-0.45 -0.28 0" />
+        <child link="link_right_back_wheel" />
+        <parent link="link_chassis" />
+        <axis rpy="0 0 0" xyz="0 1 0" />
+        <limit effort="10000" velocity="1000" />
+        <joint_properties damping="1.0" friction="1.0" />
+    </joint>
+    <link name="link_right_back_wheel">
+        <inertial>
+            <mass value="1" />
+            <origin xyz="0 0 0" rpy="0 0 0" />
+            <inertia ixx="0.002526666666667" ixy="0" ixz="0" iyy="0.002526666666667" iyz="0" izz="0.005"/>
+        </inertial>
+        <collision>
+            <origin rpy="1.5707 0 0" xyz="0 -0.18 0" />
+            <geometry>
+                <cylinder length="${length_wheel}" radius="${radius_wheel}"/>
+            </geometry>
+        </collision>
+        <visual>
+            <origin rpy="1.5707 0 0" xyz="0 -0.18 0" />
+            <geometry>
+                <cylinder length="${length_wheel}" radius="${radius_wheel}"/>
+            </geometry>
+            <material name="Black">
+                <color rgba="0.1 0.1 0.1 1" />
+            </material>
+        </visual>
+        <collision>
+            <origin rpy="1.5707 0 0" xyz="0 -0.06 0" />
+            <geometry>
+                <cylinder length="${length_cylinder_wheel}" radius="${radius_cylinder_wheel}"/>
+            </geometry>
+        </collision>
+        <visual>
+            <origin rpy="1.5707 0 0" xyz="0 -0.06 0" />
+            <geometry>
+                <cylinder length="${length_cylinder_wheel}" radius="${radius_cylinder_wheel}"/>
+            </geometry>
+            <material name="Black">
+                <color rgba="0.1 0.1 0.1 1" />
+            </material>
+        </visual>
+    </link>
+    <joint name="joint_chassis_left_front_wheel" type="continuous">
+        <origin rpy="0 0 0" xyz="0.45 0.28 0" />
+        <child link="link_left_front_wheel" />
+        <parent link="link_chassis" />
+        <axis rpy="0 0 0" xyz="0 1 0" />
+        <limit effort="10000" velocity="1000" />
+        <joint_properties damping="1.0" friction="1.0" />
+    </joint>
+    <link name="link_left_front_wheel">
+        <inertial>
+            <mass value="1" />
+            <origin xyz="0 0 0" rpy="0 0 0" />
+            <inertia ixx="0.002526666666667" ixy="0" ixz="0" iyy="0.002526666666667" iyz="0" izz="0.005"/>
+        </inertial>
+        <collision>
+            <origin rpy="1.5707 0 0" xyz="0 0.18 0" />
+            <geometry>
+                <cylinder length="${length_wheel}" radius="${radius_wheel}"/>
+            </geometry>
+        </collision>
+        <visual>
+            <origin rpy="1.5707 0 0" xyz="0 0.18 0" />
+            <geometry>
+                <cylinder length="${length_wheel}" radius="${radius_wheel}"/>
+            </geometry>
+            <material name="Black">
+                <color rgba="0.1 0.1 0.1 1" />
+            </material>
+        </visual>
+        <collision>
+            <origin rpy="1.5707 0 0" xyz="0 0.06 0" />
+            <geometry>
+                <cylinder length="${length_cylinder_wheel}" radius="${radius_cylinder_wheel}"/>
+            </geometry>
+        </collision>
+        <visual>
+            <origin rpy="1.5707 0 0" xyz="0 0.06 0" />
+            <geometry>
+                <cylinder length="${length_cylinder_wheel}" radius="${radius_cylinder_wheel}"/>
+            </geometry>
+            <material name="Black">
+                <color rgba="0.1 0.1 0.1 1" />
+            </material>
+        </visual>
+    </link>
+    <joint name="joint_chassis_right_front_wheel" type="continuous">
+        <origin rpy="0 0 0" xyz="0.45 -0.28 0" />
+        <child link="link_right_front_wheel" />
+        <parent link="link_chassis" />
+        <axis rpy="0 0 0" xyz="0 1 0" />
+        <limit effort="10000" velocity="1000" />
+        <joint_properties damping="1.0" friction="1.0" />
+    </joint>
+    <link name="link_right_front_wheel">
+        <inertial>
+            <mass value="1" />
+            <origin xyz="0 0 0" rpy="0 0 0" />
+            <inertia ixx="0.002526666666667" ixy="0" ixz="0" iyy="0.002526666666667" iyz="0" izz="0.005"/>
+        </inertial>
+        <collision>
+            <origin rpy="1.5707 0 0" xyz="0 -0.18 0" />
+            <geometry>
+                <cylinder length="${length_wheel}" radius="${radius_wheel}"/>
+            </geometry>
+        </collision>
+        <visual>
+            <origin rpy="1.5707 0 0" xyz="0 -0.18 0" />
+            <geometry>
+                <cylinder length="${length_wheel}" radius="${radius_wheel}"/>
+            </geometry>
+            <material name="Black">
+                <color rgba="0.1 0.1 0.1 1" />
+            </material>
+        </visual>
+        <collision>
+            <origin rpy="1.5707 0 0" xyz="0 -0.06 0" />
+            <geometry>
+                <cylinder length="${length_cylinder_wheel}" radius="${radius_cylinder_wheel}"/>
+            </geometry>
+        </collision>
+        <visual>
+            <origin rpy="1.5707 0 0" xyz="0 -0.06 0" />
+            <geometry>
+                <cylinder length="${length_cylinder_wheel}" radius="${radius_cylinder_wheel}"/>
+            </geometry>
+            <material name="Black">
+                <color rgba="0.1 0.1 0.1 1" />
             </material>
         </visual>

Commit message: Updated config for robot

File: robot_project/urdf/gazebo.xacro (robot description, xacro)
@@ -66,5 +66,5 @@
                 <range>
                     <min>0.20</min>
-                    <max>80.0</max>
+                    <max>12.0</max>
                     <resolution>0.01</resolution>
                 </range>

File: robot_project/urdf/robot.xacro (robot description, xacro)
@@ -218,5 +218,5 @@
     <!-- Laser scan -->
     <joint name="joint_laser_scan_chassis" type="fixed">
-        <origin rpy="0 0 0" xyz="0.4 0 0.3" />
+        <origin rpy="0 0 0" xyz="0.4 0 0.2" />
         <child link="link_laser_scan" />
         <parent link="link_chassis" />
