Commit message: Modified the robot wheels and added ekf localization

File: robot_project/urdf/gazebo.xacro (robot description, xacro)
@@ -31,9 +31,9 @@
         <plugin filename="libgazebo_ros_diff_drive.so" name="differential_drive_controller">
             <alwaysOn>true</alwaysOn>
-            <updateRate>20</updateRate>
+            <updateRate>30</updateRate>
             <leftJoint>joint_chassis_left_back_wheel</leftJoint>
             <rightJoint>joint_chassis_right_back_wheel</rightJoint>
-            <wheelSeparation>1.66</wheelSeparation>
-            <wheelDiameter>0.8</wheelDiameter>
+            <wheelSeparation>0.6</wheelSeparation>
+            <wheelDiameter>0.3</wheelDiameter>
             <torque>10</torque>
             <commandTopic>cmd_vel</commandTopic>

File: robot_project/urdf/robot.xacro (robot description, xacro)
@@ -5,7 +5,7 @@
     <xacro:property name="chassis_mass" value="10" />
     <xacro:property name="radius_wheel" value="0.15" />
-    <xacro:property name="length_wheel" value="0.12" />
+    <xacro:property name="length_wheel" value="0.06" />
     <xacro:property name="radius_cylinder_wheel" value="0.04" />
-    <xacro:property name="length_cylinder_wheel" value="0.12" />
+    <xacro:property name="length_cylinder_wheel" value="0.06" />
     <!-- Gazebo tags - Laser scan -->
     <gazebo reference="joint_laser_scan_chassis">
@@ -51,26 +51,26 @@
         </inertial>
         <collision>
-            <origin rpy="1.5707 0 0" xyz="0 0.18 0" />
-            <geometry>
-                <cylinder length="${length_wheel}" radius="${radius_wheel}"/>
-            </geometry>
-        </collision>
-        <visual>
-            <origin rpy="1.5707 0 0" xyz="0 0.18 0" />
-            <geometry>
-                <cylinder length="${length_wheel}" radius="${radius_wheel}"/>
-            </geometry>
-            <material name="Black">
-                <color rgba="0.1 0.1 0.1 1" />
-            </material>
-        </visual>
-        <collision>
-            <origin rpy="1.5707 0 0" xyz="0 0.06 0" />
-            <geometry>
-                <cylinder length="${length_cylinder_wheel}" radius="${radius_cylinder_wheel}"/>
-            </geometry>
-        </collision>
-        <visual>
-            <origin rpy="1.5707 0 0" xyz="0 0.06 0" />
+            <origin rpy="1.5707 0 0" xyz="0 0.06 0" />
+            <geometry>
+                <cylinder length="${length_wheel}" radius="${radius_wheel}"/>
+            </geometry>
+        </collision>
+        <visual>
+            <origin rpy="1.5707 0 0" xyz="0 0.06 0" />
+            <geometry>
+                <cylinder length="${length_wheel}" radius="${radius_wheel}"/>
+            </geometry>
+            <material name="Black">
+                <color rgba="0.1 0.1 0.1 1" />
+            </material>
+        </visual>
+        <collision>
+            <origin rpy="1.5707 0 0" xyz="0 0.05 0" />
+            <geometry>
+                <cylinder length="${length_cylinder_wheel}" radius="${radius_cylinder_wheel}"/>
+            </geometry>
+        </collision>
+        <visual>
+            <origin rpy="1.5707 0 0" xyz="0 0.05 0" />
             <geometry>
                 <cylinder length="${length_cylinder_wheel}" radius="${radius_cylinder_wheel}"/>
@@ -96,26 +96,26 @@
         </inertial>
         <collision>
-            <origin rpy="1.5707 0 0" xyz="0 -0.18 0" />
-            <geometry>
-                <cylinder length="${length_wheel}" radius="${radius_wheel}"/>
-            </geometry>
-        </collision>
-        <visual>
-            <origin rpy="1.5707 0 0" xyz="0 -0.18 0" />
-            <geometry>
-                <cylinder length="${length_wheel}" radius="${radius_wheel}"/>
-            </geometry>
-            <material name="Black">
-                <color rgba="0.1 0.1 0.1 1" />
-            </material>
-        </visual>
-        <collision>
-            <origin rpy="1.5707 0 0" xyz="0 -0.06 0" />
-            <geometry>
-                <cylinder length="${length_cylinder_wheel}" radius="${radius_cylinder_wheel}"/>
-            </geometry>
-        </collision>
-        <visual>
-            <origin rpy="1.5707 0 0" xyz="0 -0.06 0" />
+            <origin rpy="1.5707 0 0" xyz="0 -0.06 0" />
+            <geometry>
+                <cylinder length="${length_wheel}" radius="${radius_wheel}"/>
+            </geometry>
+        </collision>
+        <visual>
+            <origin rpy="1.5707 0 0" xyz="0 -0.06 0" />
+            <geometry>
+                <cylinder length="${length_wheel}" radius="${radius_wheel}"/>
+            </geometry>
+            <material name="Black">
+                <color rgba="0.1 0.1 0.1 1" />
+            </material>
+        </visual>
+        <collision>
+            <origin rpy="1.5707 0 0" xyz="0 -0.05 0" />
+            <geometry>
+                <cylinder length="${length_cylinder_wheel}" radius="${radius_cylinder_wheel}"/>
+            </geometry>
+        </collision>
+        <visual>
+            <origin rpy="1.5707 0 0" xyz="0 -0.05 0" />
             <geometry>
                 <cylinder length="${length_cylinder_wheel}" radius="${radius_cylinder_wheel}"/>
@@ -141,26 +141,26 @@
         </inertial>
         <collision>
-            <origin rpy="1.5707 0 0" xyz="0 0.18 0" />
-            <geometry>
-                <cylinder length="${length_wheel}" radius="${radius_wheel}"/>
-            </geometry>
-        </collision>
-        <visual>
-            <origin rpy="1.5707 0 0" xyz="0 0.18 0" />
-            <geometry>
-                <cylinder length="${length_wheel}" radius="${radius_wheel}"/>
-            </geometry>
-            <material name="Black">
-                <color rgba="0.1 0.1 0.1 1" />
-            </material>
-        </visual>
-        <collision>
-            <origin rpy="1.5707 0 0" xyz="0 0.06 0" />
-            <geometry>
-                <cylinder length="${length_cylinder_wheel}" radius="${radius_cylinder_wheel}"/>
-            </geometry>
-        </collision>
-        <visual>
-            <origin rpy="1.5707 0 0" xyz="0 0.06 0" />
+            <origin rpy="1.5707 0 0" xyz="0 0.06 0" />
+            <geometry>
+                <cylinder length="${length_wheel}" radius="${radius_wheel}"/>
+            </geometry>
+        </collision>
+        <visual>
+            <origin rpy="1.5707 0 0" xyz="0 0.06 0" />
+            <geometry>
+                <cylinder length="${length_wheel}" radius="${radius_wheel}"/>
+            </geometry>
+            <material name="Black">
+                <color rgba="0.1 0.1 0.1 1" />
+            </material>
+        </visual>
+        <collision>
+            <origin rpy="1.5707 0 0" xyz="0 0.05 0" />
+            <geometry>
+                <cylinder length="${length_cylinder_wheel}" radius="${radius_cylinder_wheel}"/>
+            </geometry>
+        </collision>
+        <visual>
+            <origin rpy="1.5707 0 0" xyz="0 0.05 0" />
             <geometry>
                 <cylinder length="${length_cylinder_wheel}" radius="${radius_cylinder_wheel}"/>
@@ -186,26 +186,26 @@
         </inertial>
         <collision>
-            <origin rpy="1.5707 0 0" xyz="0 -0.18 0" />
-            <geometry>
-                <cylinder length="${length_wheel}" radius="${radius_wheel}"/>
-            </geometry>
-        </collision>
-        <visual>
-            <origin rpy="1.5707 0 0" xyz="0 -0.18 0" />
-            <geometry>
-                <cylinder length="${length_wheel}" radius="${radius_wheel}"/>
-            </geometry>
-            <material name="Black">
-                <color rgba="0.1 0.1 0.1 1" />
-            </material>
-        </visual>
-        <collision>
-            <origin rpy="1.5707 0 0" xyz="0 -0.06 0" />
-            <geometry>
-                <cylinder length="${length_cylinder_wheel}" radius="${radius_cylinder_wheel}"/>
-            </geometry>
-        </collision>
-        <visual>
-            <origin rpy="1.5707 0 0" xyz="0 -0.06 0" />
+            <origin rpy="1.5707 0 0" xyz="0 -0.06 0" />
+            <geometry>
+                <cylinder length="${length_wheel}" radius="${radius_wheel}"/>
+            </geometry>
+        </collision>
+        <visual>
+            <origin rpy="1.5707 0 0" xyz="0 -0.06 0" />
+            <geometry>
+                <cylinder length="${length_wheel}" radius="${radius_wheel}"/>
+            </geometry>
+            <material name="Black">
+                <color rgba="0.1 0.1 0.1 1" />
+            </material>
+        </visual>
+        <collision>
+            <origin rpy="1.5707 0 0" xyz="0 -0.05 0" />
+            <geometry>
+                <cylinder length="${length_cylinder_wheel}" radius="${radius_cylinder_wheel}"/>
+            </geometry>
+        </collision>
+        <visual>
+            <origin rpy="1.5707 0 0" xyz="0 -0.05 0" />
             <geometry>
                 <cylinder length="${length_cylinder_wheel}" radius="${radius_cylinder_wheel}"/>

Commit message: Added new controller

File: robot_project/urdf/gazebo.xacro (robot description, xacro)
@@ -24,22 +24,4 @@
         <mu1>0</mu1>
         <mu2>0</mu2>
-    </gazebo>
-    <gazebo reference="joint_chassis_caster_wheel">
-        <preserveFixedJoint>true</preserveFixedJoint>
-    </gazebo>
-    <gazebo>
-        <plugin filename="libgazebo_ros_diff_drive.so" name="differential_drive_controller">
-            <alwaysOn>true</alwaysOn>
-            <updateRate>30</updateRate>
-            <leftJoint>joint_chassis_left_back_wheel</leftJoint>
-            <rightJoint>joint_chassis_right_back_wheel</rightJoint>
-            <wheelSeparation>0.6</wheelSeparation>
-            <wheelDiameter>0.3</wheelDiameter>
-            <torque>10</torque>
-            <commandTopic>cmd_vel</commandTopic>
-            <odometryTopic>odom</odometryTopic>
-            <odometryFrame>odom</odometryFrame>
-            <robotBaseFrame>link_chassis</robotBaseFrame>
-        </plugin>
     </gazebo>
     <!-- Gazebo tags - Laser scan -->
@@ -83,7 +65,9 @@
     <!-- Control plugin -->
     <gazebo>
+        <!-- Control plugin -->
         <plugin name="gazebo_ros_control" filename="libgazebo_ros_control.so">
-            <robotNamespace>/robot</robotNamespace>
+            <robotNamespace>/my_robot</robotNamespace>
             <robotSimType>gazebo_ros_control/DefaultRobotHWSim</robotSimType>
+            <legacyModeNS>true</legacyModeNS>
         </plugin>
     </gazebo>

File: robot_project/urdf/robot.xacro (robot description, xacro)
@@ -15,4 +15,24 @@
         <material>Gazebo/DarkGrey</material>
     </gazebo>
+    <transmission name="left_wheel_transmission">
+      <type>transmission_interface/SimpleTransmission</type>
+      <joint name="joint_chassis_left_back_wheel">
+        <hardwareInterface>hardware_interface/VelocityJointInterface</hardwareInterface>
+      </joint>
+      <actuator name="left_wheel_actuator">
+        <mechanicalReduction>7</mechanicalReduction>
+        <hardwareInterface>VelocityJointInterface</hardwareInterface>
+      </actuator>
+    </transmission>
+    <transmission name="right_wheel_transmission">
+      <type>transmission_interface/SimpleTransmission</type>
+      <joint name="joint_chassis_right_back_wheel">
+        <hardwareInterface>hardware_interface/VelocityJointInterface</hardwareInterface>
+      </joint>
+      <actuator name="right_wheel_actuator">
+        <mechanicalReduction>7</mechanicalReduction>
+        <hardwareInterface>VelocityJointInterface</hardwareInterface>
+      </actuator>
+    </transmission>
     <!-- Link - chassis -->
     <link name="link_chassis">
@@ -245,3 +265,23 @@
         </collision>
     </link>
+    <transmission name="left_wheel_transmission">
+      <type>transmission_interface/SimpleTransmission</type>
+      <joint name="joint_chassis_left_back_wheel">
+        <hardwareInterface>hardware_interface/VelocityJointInterface</hardwareInterface>
+      </joint>
+      <actuator name="left_wheel_actuator">
+        <mechanicalReduction>7</mechanicalReduction>
+        <hardwareInterface>VelocityJointInterface</hardwareInterface>
+      </actuator>
+    </transmission>
+    <transmission name="right_wheel_transmission">
+      <type>transmission_interface/SimpleTransmission</type>
+      <joint name="joint_chassis_right_back_wheel">
+        <hardwareInterface>hardware_interface/VelocityJointInterface</hardwareInterface>
+      </joint>
+      <actuator name="right_wheel_actuator">
+        <mechanicalReduction>7</mechanicalReduction>
+        <hardwareInterface>VelocityJointInterface</hardwareInterface>
+      </actuator>
+    </transmission>
 </robot>

Commit message: Updated config for DWAPlannerROS

File: robot_project/urdf/gazebo.xacro (robot description, xacro)
@@ -7,11 +7,11 @@
     <gazebo reference="link_left_back_wheel">
         <material>Gazebo/Black</material>
-        <mu1>1</mu1>
-        <mu2>1</mu2>
+        <mu1>0.1</mu1>
+        <mu2>0.1</mu2>
     </gazebo>
     <gazebo reference="link_right_back_wheel">
         <material>Gazebo/Black</material>
-        <mu1>1</mu1>
-        <mu2>1</mu2>
+        <mu1>0.1</mu1>
+        <mu2>0.1</mu2>
     </gazebo>
     <gazebo reference="link_left_front_wheel">

File: robot_project/urdf/robot.xacro (robot description, xacro)
@@ -218,5 +218,5 @@
     <!-- Laser scan -->
     <joint name="joint_laser_scan_chassis" type="fixed">
-        <origin rpy="0 0 0" xyz="0.4 0 0.2" />
+        <origin rpy="0 0 0" xyz="0 0 0.2" />
         <child link="link_laser_scan" />
         <parent link="link_chassis" />

Commit message: Add camera to the robot

File: robot_project/urdf/gazebo.xacro (robot description, xacro)
@@ -78,3 +78,25 @@
         </sensor>
     </gazebo>
+    <gazebo reference="camera_link">
+        <sensor name="camera" type="camera">
+            <camera>
+                <pose> 0 0 0 0 0 0 </pose>
+                <visualize>true</visualize>
+                <update_rate>10</update_rate>
+                <horizontal_fov>1.089</horizontal_fov>
+                <image>
+                    <format>R8G8B8</format>
+                    <width>640</width>
+                    <height>480</height>
+                </image>
+                <clip>
+                    <near>0.05</near>
+                    <far>30.0</far>
+                </clip>
+            </camera>
+            <plugin name="camera_controller" filename="libgazebo_ros_camera.so">
+                <frame_name>camera_link_optical</frame_name>
+            </plugin>
+        </sensor>
+    </gazebo>
 </robot>

File: robot_project/urdf/robot.xacro (robot description, xacro)
@@ -218,5 +218,5 @@
     <!-- Laser scan -->
     <joint name="joint_laser_scan_chassis" type="fixed">
-        <origin rpy="0 0 0" xyz="0 0 0.2" />
+        <origin rpy="0 0 0" xyz="0 0 0.16" />
         <child link="link_laser_scan" />
         <parent link="link_chassis" />
@@ -245,3 +245,16 @@
         </collision>
     </link>
+    <!-- Camera -->
+    <joint name="camera_joint" type="fixed">
+        <parent link="link_chassis"/>
+        <child link="camera_link"/>
+        <origin xyz="0.45 0 0.13" rpy="0 0 0"/>
+    </joint>
+    <link name="camera_link">
+        <visual>
+            <geometry>
+                <box size="0.05 0.05 0.06"/>
+            </geometry>
+        </visual>
+    </link>
 </robot>
